File: usb_pd_exporter.kicad_sch (KiCad schematic)
At the start: 18 parts, among them J1 USB-C 2.0 Female, Q1 FDS4935A, SW1 Locking_Switch, U1 CH224K

Commit message: v1.0.1
Other:
- title: (none) -> USB PD Exporter
Changed lines of the file:
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@@
 (kicad_sch (version 20230121) (generator eeschema)
   (paper "A4")
+  (title_block
+    (title "USB PD Exporter")
+    (rev "1.0.1")
+  )
   (junction (at 220.98 55.88) (diameter 0) (color 0 0 0 0)
   )
@@
     (pin "2")
     (instances
-      (project "usb_pd_sink_power"
+      (project "usb_pd_exporter"
         (path "/a99cc065-64ac-4767-b641-118f0f2c222f"
           (reference "R4") (unit 1)
@@
     (pin "1")
     (instances
-      (project "usb_pd_sink_power"
+      (project "usb_pd_exporter"
         (path "/a99cc065-64ac-4767-b641-118f0f2c222f"
           (reference "#FLG02") (unit 1)
@@
     (pin "2")
     (instances
-      (project "usb_pd_sink_power"
+      (project "usb_pd_exporter"
         (path "/a99cc065-64ac-4767-b641-118f0f2c222f"
           (reference "R2") (unit 1)
@@
     (pin "2")
     (instances
-      (project "usb_pd_sink_power"
+      (project "usb_pd_exporter"
         (path "/a99cc065-64ac-4767-b641-118f0f2c222f"
           (reference "R5") (unit 1)
@@
     (pin "1")
     (instances
-      (project "usb_pd_sink_power"
+      (project "usb_pd_exporter"
         (path "/a99cc065-64ac-4767-b641-118f0f2c222f"
           (reference "#PWR020") (unit 1)
@@
     (pin "1")
     (instances
-      (project "usb_pd_sink_power"
+      (project "usb_pd_exporter"
         (path "/a99cc065-64ac-4767-b641-118f0f2c222f"
           (reference "#PWR015") (unit 1)
@@
     (pin "1")
     (instances
-      (project "usb_pd_sink_power"
+      (project "usb_pd_exporter"
         (path "/a99cc065-64ac-4767-b641-118f0f2c222f"
           (reference "#PWR02") (unit 1)
@@
     (pin "2")
     (instances
-      (project "usb_pd_sink_power"
+      (project "usb_pd_exporter"
         (path "/a99cc065-64ac-4767-b641-118f0f2c222f"
           (reference "CH2") (unit 1)
@@
     (pin "3")
     (instances
-      (project "usb_pd_sink_power"
+      (project "usb_pd_exporter"
         (path "/a99cc065-64ac-4767-b641-118f0f2c222f"
           (reference "JP2") (unit 1)
@@
     (pin "1")
     (instances
-      (project "usb_pd_sink_power"
+      (project "usb_pd_exporter"
         (path "/a99cc065-64ac-4767-b641-118f0f2c222f"
           (reference "#PWR011") (unit 1)
@@
     (pin "2")
     (instances
-      (project "usb_pd_sink_power"
+      (project "usb_pd_exporter"
         (path "/a99cc065-64ac-4767-b641-118f0f2c222f"
           (reference "CH1") (unit 1)
@@
     (pin "1")
     (instances
-      (project "usb_pd_sink_power"
+      (project "usb_pd_exporter"
         (path "/a99cc065-64ac-4767-b641-118f0f2c222f"
           (reference "#PWR017") (unit 1)
@@
     (pin "1")
     (instances
-      (project "usb_pd_sink_power"
+      (project "usb_pd_exporter"
         (path "/a99cc065-64ac-4767-b641-118f0f2c222f"
           (reference "#PWR013") (unit 1)
@@
     (pin "3")
     (instances
-      (project "usb_pd_sink_power"
+      (project "usb_pd_exporter"
         (path "/a99cc065-64ac-4767-b641-118f0f2c222f"
           (reference "CH4") (unit 1)
@@
     (pin "1")
     (instances
-      (project "usb_pd_sink_power"
+      (project "usb_pd_exporter"
         (path "/a99cc065-64ac-4767-b641-118f0f2c222f"
           (reference "#FLG01") (unit 1)
@@
     (pin "1")
     (instances
-      (project "usb_pd_sink_power"
+      (project "usb_pd_exporter"
         (path "/a99cc065-64ac-4767-b641-118f0f2c222f"
           (reference "#PWR08") (unit 1)
@@
     (pin "9")
     (instances
-      (project "usb_pd_sink_power"
+      (project "usb_pd_exporter"
         (path "/a99cc065-64ac-4767-b641-118f0f2c222f"
           (reference "U1") (unit 1)
@@
     (pin "1")
     (instances
-      (project "usb_pd_sink_power"
+      (project "usb_pd_exporter"
         (path "/a99cc065-64ac-4767-b641-118f0f2c222f"
           (reference "#PWR03") (unit 1)
@@
     (pin "3")
     (instances
-      (project "usb_pd_sink_power"
+      (project "usb_pd_exporter"
         (path "/a99cc065-64ac-4767-b641-118f0f2c222f"
           (reference "JP3") (unit 1)
@@
     (pin "8")
     (instances
-      (project "usb_pd_sink_power"
+      (project "usb_pd_exporter"
         (path "/a99cc065-64ac-4767-b641-118f0f2c222f"
           (reference "Q1") (unit 1)
@@
     (pin "1")
     (instances
-      (project "usb_pd_sink_power"
+      (project "usb_pd_exporter"
         (path "/a99cc065-64ac-4767-b641-118f0f2c222f"
           (reference "#PWR05") (unit 1)
@@
     (pin "1")
     (instances
-      (project "usb_pd_sink_power"
+      (project "usb_pd_exporter"
         (path "/a99cc065-64ac-4767-b641-118f0f2c222f"
           (reference "#PWR010") (unit 1)
@@
     (pin "2")
     (instances
-      (project "usb_pd_sink_power"
+      (project "usb_pd_exporter"
         (path "/a99cc065-64ac-4767-b641-118f0f2c222f"
           (reference "C1") (unit 1)
@@
     (pin "2")
     (instances
-      (project "usb_pd_sink_power"
+      (project "usb_pd_exporter"
         (path "/a99cc065-64ac-4767-b641-118f0f2c222f"
           (reference "R1") (unit 1)
@@
     (pin "1")
     (instances
-      (project "usb_pd_sink_power"
+      (project "usb_pd_exporter"
         (path "/a99cc065-64ac-4767-b641-118f0f2c222f"
           (reference "#PWR019") (unit 1)
@@
     (pin "1")
     (instances
-      (project "usb_pd_sink_power"
+      (project "usb_pd_exporter"
         (path "/a99cc065-64ac-4767-b641-118f0f2c222f"
           (reference "#PWR016") (unit 1)
@@
     (pin "1")
     (instances
-      (project "usb_pd_sink_power"
+      (project "usb_pd_exporter"
         (path "/a99cc065-64ac-4767-b641-118f0f2c222f"
           (reference "#PWR012") (unit 1)
@@
     (pin "1")
     (instances
-      (project "usb_pd_sink_power"
+      (project "usb_pd_exporter"
         (path "/a99cc065-64ac-4767-b641-118f0f2c222f"
           (reference "#PWR06") (unit 1)
@@
     (pin "2")
     (instances
-      (project "usb_pd_sink_power"
+      (project "usb_pd_exporter"
         (path "/a99cc065-64ac-4767-b641-118f0f2c222f"
           (reference "R3") (unit 1)
@@
     (pin "2")
     (instances
-      (project "usb_pd_sink_power"
+      (project "usb_pd_exporter"
         (path "/a99cc065-64ac-4767-b641-118f0f2c222f"
           (reference "C2") (unit 1)
@@
     (pin "1")
     (instances
-      (project "usb_pd_sink_power"
+      (project "usb_pd_exporter"
         (path "/a99cc065-64ac-4767-b641-118f0f2c222f"
           (reference "#PWR021") (unit 1)
@@
     (pin "1")
     (instances
-      (project "usb_pd_sink_power"
+      (project "usb_pd_exporter"
         (path "/a99cc065-64ac-4767-b641-118f0f2c222f"
           (reference "#PWR04") (unit 1)
@@
     (pin "8")
     (instances
-      (project "usb_pd_sink_power"
+      (project "usb_pd_exporter"
         (path "/a99cc065-64ac-4767-b641-118f0f2c222f"
           (reference "Q1") (unit 2)
@@
     (pin "1")
     (instances
-      (project "usb_pd_sink_power"
+      (project "usb_pd_exporter"
         (path "/a99cc065-64ac-4767-b641-118f0f2c222f"
           (reference "#PWR07") (unit 1)
@@
     (pin "1")
     (instances
-      (project "usb_pd_sink_power"
+      (project "usb_pd_exporter"
         (path "/a99cc065-64ac-4767-b641-118f0f2c222f"
           (reference "#PWR09") (unit 1)
@@
     (pin "6")
     (instances
-      (project "usb_pd_sink_power"
+      (project "usb_pd_exporter"
         (path "/a99cc065-64ac-4767-b641-118f0f2c222f"
           (reference "SW1") (unit 1)
@@
     (pin "1")
     (instances
-      (project "usb_pd_sink_power"
+      (project "usb_pd_exporter"
         (path "/a99cc065-64ac-4767-b641-118f0f2c222f"
           (reference "#PWR01") (unit 1)
@@
     (pin "2")
     (instances
-      (project "usb_pd_sink_power"
+      (project "usb_pd_exporter"
         (path "/a99cc065-64ac-4767-b641-118f0f2c222f"
           (reference "CH3") (unit 1)
@@
     (pin "6")
     (instances
-      (project "usb_pd_sink_power"
+      (project "usb_pd_exporter"
         (path "/a99cc065-64ac-4767-b641-118f0f2c222f"
           (reference "J1") (unit 1)
@@
     (pin "1")
     (instances
-      (project "usb_pd_sink_power"
+      (project "usb_pd_exporter"
         (path "/a99cc065-64ac-4767-b641-118f0f2c222f"
           (reference "#PWR018") (unit 1)
@@
     (pin "3")
     (instances
-      (project "usb_pd_sink_power"
+      (project "usb_pd_exporter"
         (path "/a99cc065-64ac-4767-b641-118f0f2c222f"
           (reference "JP1") (unit 1)
